File: KiCad/DRV8876 Breakout.kicad_pcb (KiCad board)
At the start: 2 copper layers, 40.6 x 40.6 mm, 12 parts, among them J1 Conn_01x08, J2 Conn_01x08, U1 DRV8876

Commit message: Finished Schematic and PCB
Parts:
- added C6: 470uF, Capacitor_SMD:CP_Elec_10x10.5, F.Cu at (159.0, 89.3)
- added D1: KT-0603W White, LED_SMD:LED_0603_1608Metric, F.Cu at (144.6, 64.3)
- added JP1: Vref Jumper, Jumper:SolderJumper-3_P2.0mm_Open_TrianglePad1.0x1.5mm_NumberLabels, F.Cu at (140.8, 70.0)
- added JP2: PMODE Jumper, Jumper:SolderJumper-3_P2.0mm_Open_TrianglePad1.0x1.5mm_NumberLabels, F.Cu at (158.3, 67.0)
- added R5: R_Small, Resistor_SMD:R_0603_1608Metric, F.Cu at (141.0, 77.5)
- added R6: 0R, Resistor_SMD:R_0603_1608Metric, F.Cu at (141.0, 86.4)
- added R7: 1k6, Resistor_SMD:R_0603_1608Metric, F.Cu at (141.0, 83.8)
- C2, C4: value 100nF -> 22nF
- C3: value 22nF -> 100nF
- C5: value 470uF -> 100nF; footprint Capacitor_SMD:CP_Elec_10x10.5 -> Capacitor_SMD:C_0603_1608Metric
- R2: value R_Small -> 1k
- R3: value R_Small -> 10k
- moved R2 14.8 mm to (145.2, 66.8)
- moved R1 13.4 mm to (145.2, 61.8), turned to 0 degrees
- moved R4 13.0 mm to (141.0, 74.0), turned to 180 degrees
- moved C2 12.3 mm to (141.0, 82.0), turned to 180 degrees
- moved C5 12.1 mm to (150.8, 83.3)
- moved R3 11.2 mm to (141.0, 72.3), turned to 180 degrees
- moved J1 10.2 mm to (156.2, 58.4)
- moved C4 9.41 mm to (150.8, 79.0), turned to 90 degrees
- moved C1 7.16 mm to (141.0, 75.8)
- moved U1 5.08 mm to (147.3, 81.3)
- moved C3 3.81 mm to (152.6, 81.8)
Connections:
- C2 pad 1: /VM -> /IPROPI
- C2 pad 2: Net-(C2-Pad2) -> GND
- C3 pad 1: Net-(C3-Pad1) -> /VM
- C3 pad 2: Net-(C3-Pad2) -> /VCP
- C4 pad 1: /VM -> /CPH
- C4 pad 2: GND -> /CPL
- J1 pad 1: unconnected-(J1-Pad1) -> +3V3
- J1 pad 2: unconnected-(J1-Pad2) -> /EN/IN1
- J1 pad 3: unconnected-(J1-Pad3) -> /PH/IN2
- J1 pad 4: unconnected-(J1-Pad4) -> /nSLEEP
- J1 pad 5: unconnected-(J1-Pad5) -> /nFAULT
- J1 pad 6: unconnected-(J1-Pad6) -> /VREF DAC In
- J1 pad 7: unconnected-(J1-Pad7) -> /IPROPI
- J1 pad 8: unconnected-(J1-Pad8) -> /IMODE
- R1 pad 1: unconnected-(R1-Pad1) -> +3V3
- R1 pad 2: /VREF -> /nFAULT
- R2 pad 1: /VM -> /LED K
- R2 pad 2: /VREF -> /nFAULT
- R3 pad 1: /VREF -> /VREF Jumper
- R3 pad 2: GND -> /VREF
- R4 pad 1: unconnected-(R4-Pad1) -> +3V3
- R4 pad 2: unconnected-(R4-Pad2) -> /VREF
- U1 pad 1: unconnected-(U1-Pad1) -> /nSLEEP
- U1 pad 10: Net-(C2-Pad2) -> /VCP
- U1 pad 11: Net-(C3-Pad1) -> /CPH
- U1 pad 12: Net-(C3-Pad2) -> /CPL
- U1 pad 14: unconnected-(U1-Pad14) -> /PMODE
- U1 pad 15: unconnected-(U1-Pad15) -> /EN/IN1
- U1 pad 16: unconnected-(U1-Pad16) -> /PH/IN2
- U1 pad 2: unconnected-(U1-Pad2) -> /nFAULT
- U1 pad 3: unconnected-(U1-Pad3) -> /VREF
- U1 pad 4: unconnected-(U1-Pad4) -> /IPROPI
- U1 pad 5: unconnected-(U1-Pad5) -> /IMODE
Routing:
- net /IMODE: track 0.00 -> 43.2 mm
- net +3V3: track 0.00 -> 40.1 mm
- net /IPROPI: track 0.00 -> 33.2 mm
- net /VM: track 0.00 -> 30.6 mm
- net /nFAULT: track 0.00 -> 26.1 mm
- net /nSLEEP: track 0.00 -> 25.0 mm
- net /EN/IN1: track 0.00 -> 24.2 mm
- net /PH/IN2: track 0.00 -> 23.3 mm
- net /PMODE: track 0.00 -> 19.6 mm
- net GND: track 0.00 -> 18.8 mm, vias 0 -> 33
- net /VREF DAC In: track 0.00 -> 13.5 mm
- net /VREF: track 0.00 -> 13.5 mm
- net /OUT2: track 0.00 -> 5.30 mm
- net /OUT1: track 0.00 -> 5.10 mm
- net /VCP: track 0.00 -> 4.08 mm
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- added copper zone on F.Cu, net /OUT1
- added copper zone on F.Cu, net /OUT2
- added copper zone on F.Cu, net /VM
Other:
- board size 40.6 x 40.6 mm -> 38.1 x 50.8 mm

Commit message: Finished and Plotted
Parts:
- added REF**: Logo, MEPOS:Logo, F.Cu at (147.3, 66.0)
- added kibuzzard-633DB2C4: G***, kibuzzard-633DB2C4, F.Cu at (137.2, 90.2)
- added kibuzzard-633DB2E1: G***, kibuzzard-633DB2E1, F.Cu at (137.2, 92.7)
- added kibuzzard-633DB301: G***, kibuzzard-633DB301, F.Cu at (137.2, 95.2)
- added kibuzzard-633DB48A: G***, kibuzzard-633DB48A, F.Cu at (158.1, 69.2)
- added kibuzzard-633DB49D: G***, kibuzzard-633DB49D, F.Cu at (136.7, 68.4)
- moved R1 6.53 mm to (143.3, 68.0)
- moved R2 6.53 mm to (143.3, 73.0)
- moved D1 6.53 mm to (142.6, 70.5)
- moved JP2 5.08 mm to (158.3, 72.1)
- moved C1 3.82 mm to (137.4, 76.9)
- moved JP1 3.82 mm to (137.2, 71.1)
- moved R3 3.82 mm to (137.3, 73.4)
- moved R4 3.82 mm to (137.3, 75.1)
- moved R5 3.82 mm to (137.3, 78.6)
Routing:
- net /OUT1: track 5.10 -> 24.9 mm
- net /OUT2: track 5.30 -> 24.4 mm
- net +3V3: track 40.1 -> 50.1 mm
- net /IPROPI: track 33.2 -> 40.5 mm
- net /IMODE: track 43.2 -> 49.1 mm
- net /PMODE: track 19.6 -> 15.3 mm
- net /VREF DAC In: track 13.5 -> 16.2 mm
- net /VREF: track 13.5 -> 15.4 mm
- net /nFAULT: track 26.1 -> 25.3 mm
- net GND: vias 33 -> 48
Other:
- board text added: "+3V3"
- board text added: "EN/IN1"
- board text added: "GND"
- board text added: "IMODE"
- board text added: "IPROPI"
- board text added: "JLCJLCJLCJLC"
- board text added: "OUT1"
- board text added: "OUT2"
- board text added: "PH/IN2"
- board text added: "VM"
- board text added: "VREF IN"
- board text added: "nFAULT"
- board text added: "nSLEEP"

Commit message: Update DRV8876 Breakout.kicad_pcb
Parts:
- C6: value 470uF -> 220uF
- D1: value KT-0603W White -> 0603 Red
- R4, R5: value R_Small -> NF
Changed lines of the file:
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@@
     (descr "Capacitor SMD 0603 (1608 Metric), square (rectangular) end terminal, IPC_7351 nominal, (Body size source: IPC-SM-782 page 76, https://www.pcb-3d.com/wordpress/wp-content/uploads/ipc-sm-782a_amendment_1_and_2.pdf), generated with kicad-footprint-generator")
     (tags "capacitor")
+    (property "MFR Number" "GRM188R61C106MAALD")
+    (property "Mouser Part Number" "81-GRM188R61C106MALD")
     (property "Sheetfile" "DRV8876 Breakout.kicad_sch")
     (property "Sheetname" "")
@@
     (descr "Resistor SMD 0603 (1608 Metric), square (rectangular) end terminal, IPC_7351 nominal, (Body size source: IPC-SM-782 page 72, https://www.pcb-3d.com/wordpress/wp-content/uploads/ipc-sm-782a_amendment_1_and_2.pdf), generated with kicad-footprint-generator")
     (tags "resistor")
+    (property "MFR Number" "")
+    (property "Mouser Part Number" "")
     (property "Sheetfile" "DRV8876 Breakout.kicad_sch")
     (property "Sheetname" "")
@@
       (effects (font (size 1 1) (thickness 0.15)))
     )
-    (fp_text value "R_Small" (at 0 1.43) (layer "F.Fab")
+    (fp_text value "NF" (at 0 1.43) (layer "F.Fab")
       (effects (font (size 1 1) (thickness 0.15)))
     )
@@
     (descr "VQFN, 16 Pin (http://www.ti.com/lit/ds/sbos354a/sbos354a.pdf, JEDEC MO-220 variant VEED-6), generated with kicad-footprint-generator ipc_noLead_generator.py")
     (tags "VQFN NoLead")
+    (property "MFR Number" "DRV8876RGTR")
+    (property "Mouser Part Number" "595-DRV8876RGTR")
     (property "Sheetfile" "DRV8876 Breakout.kicad_sch")
     (property "Sheetname" "")
@@
     (descr "Capacitor SMD 0603 (1608 Metric), square (rectangular) end terminal, IPC_7351 nominal, (Body size source: IPC-SM-782 page 76, https://www.pcb-3d.com/wordpress/wp-content/uploads/ipc-sm-782a_amendment_1_and_2.pdf), generated with kicad-footprint-generator")
     (tags "capacitor")
+    (property "MFR Number" "06035C104KAZ4A")
+    (property "Mouser Part Number" "581-06035C104KAZ4A")
     (property "Sheetfile" "DRV8876 Breakout.kicad_sch")
     (property "Sheetname" "")
@@
     (descr "Resistor SMD 0603 (1608 Metric), square (rectangular) end terminal, IPC_7351 nominal, (Body size source: IPC-SM-782 page 72, https://www.pcb-3d.com/wordpress/wp-content/uploads/ipc-sm-782a_amendment_1_and_2.pdf), generated with kicad-footprint-generator")
     (tags "resistor")
+    (property "MFR Number" "RK73Z1JTTD")
+    (property "Mouser Part Number" "660-RK73Z1JTTD")
     (property "Sheetfile" "DRV8876 Breakout.kicad_sch")
     (property "Sheetname" "")
@@
     (descr "Resistor SMD 0603 (1608 Metric), square (rectangular) end terminal, IPC_7351 nominal, (Body size source: IPC-SM-782 page 72, https://www.pcb-3d.com/wordpress/wp-content/uploads/ipc-sm-782a_amendment_1_and_2.pdf), generated with kicad-footprint-generator")
     (tags "resistor")
+    (property "MFR Number" "ERA-3AEB162V")
+    (property "Mouser Part Number" "667-ERA-3AEB162V")
     (property "Sheetfile" "DRV8876 Breakout.kicad_sch")
     (property "Sheetname" "")
@@
     (descr "Resistor SMD 0603 (1608 Metric), square (rectangular) end terminal, IPC_7351 nominal, (Body size source: IPC-SM-782 page 72, https://www.pcb-3d.com/wordpress/wp-content/uploads/ipc-sm-782a_amendment_1_and_2.pdf), generated with kicad-footprint-generator")
     (tags "resistor")
+    (property "MFR Number" "CR0603AFX-1001EAS")
+    (property "Mouser Part Number" "652-CR0603AFX1001EAS")
     (property "Sheetfile" "DRV8876 Breakout.kicad_sch")
     (property "Sheetname" "")
@@
     (descr "Capacitor SMD 0603 (1608 Metric), square (rectangular) end terminal, IPC_7351 nominal, (Body size source: IPC-SM-782 page 76, https://www.pcb-3d.com/wordpress/wp-content/uploads/ipc-sm-782a_amendment_1_and_2.pdf), generated with kicad-footprint-generator")
     (tags "capacitor")
+    (property "MFR Number" "GCJ188R71H223KA01D")
+    (property "Mouser Part Number" "81-GCJ188R71H223KA1D")
     (property "Sheetfile" "DRV8876 Breakout.kicad_sch")
     (property "Sheetname" "")
@@
     (descr "LED SMD 0603 (1608 Metric), square (rectangular) end terminal, IPC_7351 nominal, (Body size source: http://www.tortai-tech.com/upload/download/2011102023233369053.pdf), generated with kicad-footprint-generator")
     (tags "LED")
+    (property "MFR Number" "150060RS75000")
+    (property "Mouser Part Number" "710-150060RS75000")
     (property "Sheetfile" "DRV8876 Breakout.kicad_sch")
     (property "Sheetname" "")
@@
       (effects (font (size 1 1) (thickness 0.15)))
     )
-    (fp_text value "KT-0603W White" (at 0 1.43 90) (layer "F.Fab")
+    (fp_text value "0603 Red" (at 0 1.43 90) (layer "F.Fab")
       (effects (font (size 1 1) (thickness 0.15)))
     )
@@
     )
   )
-  (footprint "MEPOS:Logo" (layer "F.Cu")
+  (footprint "MEPOS:Logo" locked (layer "F.Cu")
     (at 147.32 66.04)
     (attr smd)
@@
     (descr "Resistor SMD 0603 (1608 Metric), square (rectangular) end terminal, IPC_7351 nominal, (Body size source: IPC-SM-782 page 72, https://www.pcb-3d.com/wordpress/wp-content/uploads/ipc-sm-782a_amendment_1_and_2.pdf), generated with kicad-footprint-generator")
     (tags "resistor")
+    (property "MFR Number" "AC0603FR-1010KL")
+    (property "Mouser Part Number" "603-AC0603FR-1010KL")
     (property "Sheetfile" "DRV8876 Breakout.kicad_sch")
     (property "Sheetname" "")
@@
     (descr "Capacitor SMD 0603 (1608 Metric), square (rectangular) end terminal, IPC_7351 nominal, (Body size source: IPC-SM-782 page 76, https://www.pcb-3d.com/wordpress/wp-content/uploads/ipc-sm-782a_amendment_1_and_2.pdf), generated with kicad-footprint-generator")
     (tags "capacitor")
+    (property "MFR Number" "GCJ188R71H223KA01D")
+    (property "Mouser Part Number" "81-GCJ188R71H223KA1D")
     (property "Sheetfile" "DRV8876 Breakout.kicad_sch")
     (property "Sheetname" "")
@@
     (property "Sheetfile" "DRV8876 Breakout.kicad_sch")
     (property "Sheetname" "")
-    (attr exclude_from_pos_files)
+    (property "exclude_from_bom" "")
+    (attr exclude_from_pos_files exclude_from_bom)
     (fp_text reference "JP1" (at -3.025 2.36) (layer "F.SilkS")
       (effects (font (size 1 1) (thickness 0.15)))
@@
     (descr "SMD capacitor, aluminum electrolytic, Vishay 1010, 10.0x10.5mm, http://www.vishay.com/docs/28395/150crz.pdf")
     (tags "capacitor electrolytic")
+    (property "MFR Number" "EDK227M050A9PAA")
+    (property "Mouser Part Number" "80-EDK227M050A9PAA")
     (property "Sheetfile" "DRV8876 Breakout.kicad_sch")
     (property "Sheetname" "")
@@
       (effects (font (size 1 1) (thickness 0.15)))
     )
-    (fp_text value "470uF" (at 0 6.3) (layer "F.Fab")
+    (fp_text value "220uF" (at 0 6.3) (layer "F.Fab")
       (effects (font (size 1 1) (thickness 0.15)))
     )
@@
     (property "Sheetfile" "DRV8876 Breakout.kicad_sch")
     (property "Sheetname" "")
-    (attr exclude_from_pos_files)
+    (property "exclude_from_bom" "")
+    (attr exclude_from_pos_files exclude_from_bom)
     (fp_text reference "JP2" (at 0 -2.25) (layer "F.SilkS")
       (effects (font (size 1 1) (thickness 0.15)))
@@
     (descr "Capacitor SMD 0603 (1608 Metric), square (rectangular) end terminal, IPC_7351 nominal, (Body size source: IPC-SM-782 page 76, https://www.pcb-3d.com/wordpress/wp-content/uploads/ipc-sm-782a_amendment_1_and_2.pdf), generated with kicad-footprint-generator")
     (tags "capacitor")
+    (property "MFR Number" "06035C104KAZ4A")
+    (property "Mouser Part Number" "581-06035C104KAZ4A")
     (property "Sheetfile" "DRV8876 Breakout.kicad_sch")
     (property "Sheetname" "")
@@
     (descr "Resistor SMD 0603 (1608 Metric), square (rectangular) end terminal, IPC_7351 nominal, (Body size source: IPC-SM-782 page 72, https://www.pcb-3d.com/wordpress/wp-content/uploads/ipc-sm-782a_amendment_1_and_2.pdf), generated with kicad-footprint-generator")
     (tags "resistor")
+    (property "MFR Number" "")
+    (property "Mouser Part Number" "")
     (property "Sheetfile" "DRV8876 Breakout.kicad_sch")
     (property "Sheetname" "")
@@
       (effects (font (size 1 1) (thickness 0.15)))
     )
-    (fp_text value "R_Small" (at 0 1.43) (layer "F.Fab")
+    (fp_text value "NF" (at 0 1.43) (layer "F.Fab")
       (effects (font (size 1 1) (thickness 0.15)))
     )
@@
     (descr "Resistor SMD 0603 (1608 Metric), square (rectangular) end terminal, IPC_7351 nominal, (Body size source: IPC-SM-782 page 72, https://www.pcb-3d.com/wordpress/wp-content/uploads/ipc-sm-782a_amendment_1_and_2.pdf), generated with kicad-footprint-generator")
     (tags "resistor")
+    (property "MFR Number" "AC0603FR-1010KL")
+    (property "Mouser Part Number" "603-AC0603FR-1010KL")
     (property "Sheetfile" "DRV8876 Breakout.kicad_sch")
     (property "Sheetname" "")
@@
     (descr "Through hole straight pin header, 1x08, 2.54mm pitch, single row")
     (tags "Through hole pin header THT 1x08 2.54mm single row")
+    (property "MFR Number" "10129378-908001BLF")
+    (property "Mouser Part Number" "649-1012937890801BLF")
     (property "Sheetfile" "DRV8876 Breakout.kicad_sch")
     (property "Sheetname" "")
@@
     (descr "Through hole straight pin header, 1x08, 2.54mm pitch, single row")
     (tags "Through hole pin header THT 1x08 2.54mm single row")
+    (property "MFR Number" "10129378-908001BLF")
+    (property "Mouser Part Number" "649-1012937890801BLF")
     (property "Sheetfile" "DRV8876 Breakout.kicad_sch")
     (property "Sheetname" "")
