File: KiCad/DRV8876 Breakout.kicad_sch (KiCad schematic)
At the start: 12 parts, among them J1 Conn_01x08, J2 Conn_01x08, U1 DRV8876

Commit message: Finished Schematic and PCB
Parts:
- added C2: 22nF, Capacitor_SMD:C_0603_1608Metric, symbol Device:C_Small
- added D1: KT-0603W White, LED_SMD:LED_0603_1608Metric, symbol Device:LED_Small
- added JP1: Vref Jumper, Jumper:SolderJumper-3_P2.0mm_Open_TrianglePad1.0x1.5mm_NumberLabels, symbol Jumper:SolderJumper_3_Open
- added JP2: PMODE Jumper, Jumper:SolderJumper-3_P2.0mm_Open_TrianglePad1.0x1.5mm_NumberLabels, symbol Jumper:SolderJumper_3_Open
- added R1: 10k, Resistor_SMD:R_0603_1608Metric, symbol Device:R_Small
- added R2: 1k, Resistor_SMD:R_0603_1608Metric, symbol Device:R_Small
- added R6: 0R, Resistor_SMD:R_0603_1608Metric, symbol Device:R_Small
- R7: renamed from R4; value R_Small -> 1k6
- renumbered C2 to C3, C3 to C4, C4 to C5, C5 to C6, R1 to R3, R2 to R4, R3 to R5
Connections:
- net GND: now also R7.2, C2.2, JP2.1 (A), R6.2
- net VM: no longer R4.1
- net VREF: now also U1.3 (VREF)
- net nSLEEP: now reaches U1.1 (nSLEEP)
- net nSLEEP: now also J1.4 (Pin_4)
- net VCP: now reaches C3.2, U1.10 (VCP)
- net CPH: now reaches C4.1, U1.11 (CPH)
- net CPL: now reaches C4.2, U1.12 (CPL)
- net PMODE: now reaches U1.14 (PMODE)
- net PMODE: now also JP2.2 (C)
- net EN/IN1: now reaches U1.15 (EN/IN1)
- net EN/IN1: now also J1.2 (Pin_2)
- net PH/IN2: now reaches U1.16 (PH/IN2)
- net PH/IN2: now also J1.3 (Pin_3)
- net nFAULT: now reaches U1.2 (nFAULT)
- net nFAULT: now also J1.5 (Pin_5), R1.2, R2.2
- net IPROPI: now reaches U1.4 (IPROPI)
- net IPROPI: now also J1.7 (Pin_7), R7.1, C2.1
- net IMODE: now reaches U1.5 (IMODE)
- net IMODE: now also J1.8 (Pin_8), R6.1
- net +3V3: now reaches J1.1 (Pin_1)
- net +3V3: now also R4.1, D1.2 (A), JP1.3 (B), JP2.3 (B), R1.1
- net VREF DAC In: now reaches J1.6 (Pin_6)
- net VREF DAC In: now also JP1.1 (A)
- net VREF Jumper: now reaches R3.1
- net VREF Jumper: now also JP1.2 (C)
- new net LED K: D1.1 (K), R2.1
Other:
- note added: "Ipropi(uA) = (Ils2 + Ils1)(A) * Aipropi(uA/A) Vipropi = Ipropi * Ripropi Imax = 2A Aipropi = 1000(uA/A) Ipropi = 2 * 1000 = 2000 (uA) Vadc = 3.3V 3.3 / 0.002 = 1650 Ripropi = 1k6"
- note added: "Itrip * Aipropi(uA/A) = Vvref / Ripropi Itrip * 0.001 = 3.3 / 1600 Itrip = 2.0625(A)"
- note added: "PMODE = HIGH = PH/EN Mode PMODE = LOW = PWM Mode PMODE = Hi-Z = Independant Mode Must pull nSLEEP low to change mode"
- note added: "Rimode"
- note added: "Rimode = GND = FO-T & AR Rimode = 20k = C-B-C & AR Rimode = 62k = C-B-C & OLO Rimode = Hi-Z = FO-T & OLO Must pull nSLEEP low to change mode"
- note added: "Ripropi"
- moved on the sheet: C1, C3, C4, C5, C6, J2, R3, R4, R5, R7, U1

Commit message: Update DRV8876 Breakout.kicad_sch
Parts:
- R4, R5: value R_Small -> NF
Changed lines of the file:
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@@
       (effects (font (size 1.27 1.27)) (justify left))
     )
-    (property "Value" "R_Small" (id 1) (at 129.54 66.0399 0)
+    (property "Value" "NF" (id 1) (at 129.54 66.0399 0)
       (effects (font (size 1.27 1.27)) (justify left))
     )
@@
       (effects (font (size 1.27 1.27)) (justify left))
     )
-    (property "Value" "R_Small" (id 1) (at 128.27 55.8799 0)
+    (property "Value" "NF" (id 1) (at 128.27 55.8799 0)
       (effects (font (size 1.27 1.27)) (justify left))
     )
@@
     )
     (path "/d4d0cc60-c628-4736-a572-fb065bd5d8f6"
-      (reference "R4") (unit 1) (value "R_Small") (footprint "Resistor_SMD:R_0603_1608Metric")
+      (reference "R4") (unit 1) (value "NF") (footprint "Resistor_SMD:R_0603_1608Metric")
     )
     (path "/93acd34a-27c8-4929-ab6c-4f07f49c497a"
-      (reference "R5") (unit 1) (value "R_Small") (footprint "Resistor_SMD:R_0603_1608Metric")
+      (reference "R5") (unit 1) (value "NF") (footprint "Resistor_SMD:R_0603_1608Metric")
     )
     (path "/5b5d581d-3232-4b76-a867-2637b824d46f"

Commit message: Update DRV8876 Breakout.kicad_sch
Parts:
- C1: MFR Number (none) -> GRM188R61C106MAALD; Mouser Part Number (none) -> 81-GRM188R61C106MALD
- C2, C4: MFR Number (none) -> GCJ188R71H223KA01D; Mouser Part Number (none) -> 81-GCJ188R71H223KA1D
- C3, C5: MFR Number (none) -> 06035C104KAZ4A; Mouser Part Number (none) -> 581-06035C104KAZ4A
- C6: value 470uF -> 220uF; MFR Number (none) -> EDK227M050A9PAA; Mouser Part Number (none) -> 80-EDK227M050A9PAA
- D1: value KT-0603W White -> 0603 Red; MFR Number (none) -> 150060RS75000; Mouser Part Number (none) -> 710-150060RS75000
- J1, J2: MFR Number (none) -> 10129378-908001BLF; Mouser Part Number (none) -> 649-1012937890801BLF
- JP1, JP2: now left out of the parts list
- R1, R3: MFR Number (none) -> AC0603FR-1010KL; Mouser Part Number (none) -> 603-AC0603FR-1010KL
- R2: MFR Number (none) -> CR0603AFX-1001EAS; Mouser Part Number (none) -> 652-CR0603AFX1001EAS
- R6: MFR Number (none) -> RK73Z1JTTD; Mouser Part Number (none) -> 660-RK73Z1JTTD
- R7: MFR Number (none) -> ERA-3AEB162V; Mouser Part Number (none) -> 667-ERA-3AEB162V
- U1: MFR Number (none) -> DRV8876RGTR; Mouser Part Number (none) -> 595-DRV8876RGTR
Changed lines of the file:
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@@
+      (effects (font (size 1.27 1.27)) hide)
+    )
+    (property "MFR Number" "DRV8876RGTR" (id 4) (at 190.5 101.6 0)
+      (effects (font (size 1.27 1.27)) hide)
+    )
+    (property "Mouser Part Number" "595-DRV8876RGTR" (id 5) (at 190.5 101.6 0)
       (effects (font (size 1.27 1.27)) hide)
     )
@@
   )
   (symbol (lib_id "Jumper:SolderJumper_3_Open") (at 158.75 43.18 90) (unit 1)
-    (in_bom yes) (on_board yes) (fields_autoplaced)
+    (in_bom no) (on_board yes) (fields_autoplaced)
     (property "Reference" "JP2" (id 0) (at 156.21 41.9099 90)
       (effects (font (size 1.27 1.27)) (justify left))
@@
       (effects (font (size 1.27 1.27)) hide)
     )
+    (property "MFR Number" "06035C104KAZ4A" (id 4) (at 217.17 92.71 0)
+      (effects (font (size 1.27 1.27)) hide)
+    )
+    (property "Mouser Part Number" "581-06035C104KAZ4A" (id 5) (at 217.17 92.71 0)
+      (effects (font (size 1.27 1.27)) hide)
+    )
     (pin "1")
     (pin "2")
@@
       (effects (font (size 1.27 1.27)) hide)
     )
+    (property "MFR Number" "RK73Z1JTTD" (id 4) (at 127 114.3 0)
+      (effects (font (size 1.27 1.27)) hide)
+    )
+    (property "Mouser Part Number" "660-RK73Z1JTTD" (id 5) (at 127 114.3 0)
+      (effects (font (size 1.27 1.27)) hide)
+    )
     (pin "1")
     (pin "2")
@@
     )
     (property "Datasheet" "~" (id 3) (at 254 102.87 0)
+      (effects (font (size 1.27 1.27)) hide)
+    )
+    (property "MFR Number" "10129378-908001BLF" (id 4) (at 254 102.87 0)
+      (effects (font (size 1.27 1.27)) hide)
+    )
+    (property "Mouser Part Number" "649-1012937890801BLF" (id 5) (at 254 102.87 0)
       (effects (font (size 1.27 1.27)) hide)
     )
@@
       (effects (font (size 1.27 1.27)) hide)
     )
+    (property "MFR Number" "CR0603AFX-1001EAS" (id 4) (at 96.52 85.09 0)
+      (effects (font (size 1.27 1.27)) hide)
+    )
+    (property "Mouser Part Number" "652-CR0603AFX1001EAS" (id 5) (at 96.52 85.09 0)
+      (effects (font (size 1.27 1.27)) hide)
+    )
     (pin "1")
     (pin "2")
@@
       (effects (font (size 1.27 1.27)) hide)
     )
+    (property "MFR Number" "06035C104KAZ4A" (id 4) (at 204.47 92.71 0)
+      (effects (font (size 1.27 1.27)) hide)
+    )
+    (property "Mouser Part Number" "581-06035C104KAZ4A" (id 5) (at 204.47 92.71 0)
+      (effects (font (size 1.27 1.27)) hide)
+    )
     (pin "1")
     (pin "2")
@@
       (effects (font (size 1.27 1.27)) hide)
     )
+    (property "MFR Number" "GCJ188R71H223KA01D" (id 4) (at 148.59 114.3 0)
+      (effects (font (size 1.27 1.27)) hide)
+    )
+    (property "Mouser Part Number" "81-GCJ188R71H223KA1D" (id 5) (at 148.59 114.3 0)
+      (effects (font (size 1.27 1.27)) hide)
+    )
     (pin "1")
     (pin "2")
@@
       (effects (font (size 1.27 1.27)) hide)
     )
+    (property "MFR Number" "" (id 4) (at 127 64.77 0)
+      (effects (font (size 1.27 1.27)) hide)
+    )
+    (property "Mouser Part Number" "" (id 5) (at 127 64.77 0)
+      (effects (font (size 1.27 1.27)) hide)
+    )
     (pin "1")
     (pin "2")
@@
     )
     (property "Datasheet" "~" (id 3) (at 88.9 85.09 0)
+      (effects (font (size 1.27 1.27)) hide)
+    )
+    (property "MFR Number" "AC0603FR-1010KL" (id 4) (at 88.9 85.09 0)
+      (effects (font (size 1.27 1.27)) hide)
+    )
+    (property "Mouser Part Number" "603-AC0603FR-1010KL" (id 5) (at 88.9 85.09 0)
       (effects (font (size 1.27 1.27)) hide)
     )
@@
     )
     (property "Datasheet" "~" (id 3) (at 45.72 97.79 0)
+      (effects (font (size 1.27 1.27)) hide)
+    )
+    (property "MFR Number" "10129378-908001BLF" (id 4) (at 45.72 97.79 0)
+      (effects (font (size 1.27 1.27)) hide)
+    )
+    (property "Mouser Part Number" "649-1012937890801BLF" (id 5) (at 45.72 97.79 0)
       (effects (font (size 1.27 1.27)) hide)
     )
@@
       (effects (font (size 1.27 1.27)) (justify right))
     )
-    (property "Value" "KT-0603W White" (id 1) (at 99.06 78.6764 90)
+    (property "Value" "0603 Red" (id 1) (at 99.06 78.6764 90)
       (effects (font (size 1.27 1.27)) (justify right))
     )
@@
     )
     (property "Datasheet" "~" (id 3) (at 96.52 77.47 90)
+      (effects (font (size 1.27 1.27)) hide)
+    )
+    (property "MFR Number" "150060RS75000" (id 4) (at 96.52 77.47 0)
+      (effects (font (size 1.27 1.27)) hide)
+    )
+    (property "Mouser Part Number" "710-150060RS75000" (id 5) (at 96.52 77.47 0)
       (effects (font (size 1.27 1.27)) hide)
     )
@@
       (effects (font (size 1.27 1.27)) hide)
     )
+    (property "MFR Number" "AC0603FR-1010KL" (id 4) (at 111.76 59.69 0)
+      (effects (font (size 1.27 1.27)) hide)
+    )
+    (property "Mouser Part Number" "603-AC0603FR-1010KL" (id 5) (at 111.76 59.69 0)
+      (effects (font (size 1.27 1.27)) hide)
+    )
     (pin "1")
     (pin "2")
@@
     )
     (property "Datasheet" "~" (id 3) (at 125.73 54.61 0)
+      (effects (font (size 1.27 1.27)) hide)
+    )
+    (property "MFR Number" "" (id 4) (at 125.73 54.61 0)
+      (effects (font (size 1.27 1.27)) hide)
+    )
+    (property "Mouser Part Number" "" (id 5) (at 125.73 54.61 0)
       (effects (font (size 1.27 1.27)) hide)
     )
@@
       (effects (font (size 1.27 1.27)) (justify left))
     )
-    (property "Value" "470uF" (id 1) (at 232.41 93.98 0)
+    (property "Value" "220uF" (id 1) (at 232.41 93.98 0)
       (effects (font (size 1.27 1.27)) (justify left))
     )
@@
       (effects (font (size 1.27 1.27)) hide)
     )
+    (property "MFR Number" "EDK227M050A9PAA" (id 4) (at 229.87 92.71 0)
+      (effects (font (size 1.27 1.27)) hide)
+    )
+    (property "Mouser Part Number" "80-EDK227M050A9PAA" (id 5) (at 229.87 92.71 0)
+      (effects (font (size 1.27 1.27)) hide)
+    )
     (pin "1")
     (pin "2")
@@
       (effects (font (size 1.27 1.27)) hide)
     )
+    (property "MFR Number" "ERA-3AEB162V" (id 4) (at 166.37 114.3 0)
+      (effects (font (size 1.27 1.27)) hide)
+    )
+    (property "Mouser Part Number" "667-ERA-3AEB162V" (id 5) (at 166.37 114.3 0)
+      (effects (font (size 1.27 1.27)) hide)
+    )
     (pin "1")
     (pin "2")
@@
       (effects (font (size 1.27 1.27)) hide)
     )
+    (property "MFR Number" "GCJ188R71H223KA01D" (id 4) (at 204.47 100.33 0)
+      (effects (font (size 1.27 1.27)) hide)
+    )
+    (property "Mouser Part Number" "81-GCJ188R71H223KA1D" (id 5) (at 204.47 100.33 0)
+      (effects (font (size 1.27 1.27)) hide)
+    )
     (pin "1")
     (pin "2")
   )
   (symbol (lib_id "Jumper:SolderJumper_3_Open") (at 101.6 50.8 0) (unit 1)
-    (in_bom yes) (on_board yes) (fields_autoplaced)
+    (in_bom no) (on_board yes) (fields_autoplaced)
     (property "Reference" "JP1" (id 0) (at 101.6 44.45 0))
     (property "Value" "Vref Jumper" (id 1) (at 101.6 46.99 0))
@@
       (effects (font (size 1.27 1.27)) hide)
     )
+    (property "MFR Number" "GRM188R61C106MAALD" (id 4) (at 116.84 64.77 0)
+      (effects (font (size 1.27 1.27)) hide)
+    )
+    (property "Mouser Part Number" "81-GRM188R61C106MALD" (id 5) (at 116.84 64.77 0)
+      (effects (font (size 1.27 1.27)) hide)
+    )
     (pin "1")
     (pin "2")
@@
     )
     (path "/da6ef574-5620-4a1d-af97-177792e30cd3"
-      (reference "C6") (unit 1) (value "470uF") (footprint "Capacitor_SMD:CP_Elec_10x10.5")
+      (reference "C6") (unit 1) (value "220uF") (footprint "Capacitor_SMD:CP_Elec_10x10.5")
     )
     (path "/a9d388ef-83e7-4cd9-817d-690365033f05"
-      (reference "D1") (unit 1) (value "KT-0603W White") (footprint "LED_SMD:LED_0603_1608Metric")
+      (reference "D1") (unit 1) (value "0603 Red") (footprint "LED_SMD:LED_0603_1608Metric")
     )
     (path "/a8895591-66be-432d-bdde-98f78512621f"
